Commit message: tested changes to computeinertiawrtCOM added support for CoM and frame angle

File: URDFs/kuka_kr210_payload.urdf (robot description, URDF)
Before this commit: robot kuka_kr210, 7 links, 6 joints
Joints:
- joint joint_3: type revolute -> fixed

File: URDFs/kuka_kr210_payload_env.urdf (robot description, URDF)
Before this commit: robot kuka_kr210, 7 links, 6 joints
Links:
- link link_6: mass 6.3154 -> envvar_1
Joints:
- joint joint_6: type revolute -> fixed

File: URDFs/twoLinks.urdf (robot description, URDF)
Before this commit: robot twoLinks, 3 links, 2 joints
Joints:
- joint base_fixed_joint: axis 0 0 0 -> 0 0 1; type fixed -> revolute
- joint joint_1_2: type continuous -> revolute
